File: RM_47mm.kicad_sch (KiCad schematic)
At the start: 18 parts, among them P1 USB_C_Plug, U1 STM32F103C8Tx

Commit message: 电路图初版完成
Parts:
- removed P1: USB_C_Plug, symbol Connector:USB_C_Plug
- added C10, C9: 100nf, Capacitor_SMD:C_0603_1608Metric, symbol Device:C
- added C11: 4.7uf, Capacitor_SMD:C_0603_1608Metric, symbol Device:C
- added C12: 0.1uf, Capacitor_SMD:C_0603_1608Metric, symbol Device:C
- added J1: USB_C_Receptacle_USB2.0, symbol Connector:USB_C_Receptacle_USB2.0
- added J2: SWD, Connector_JST:JST_GH_SM04B-GHS-TB_1x04-1MP_P1.25mm_Horizontal, symbol Connector:Conn_01x04_Pin
- added R1: 10k, Resistor_SMD:R_0603_1608Metric, symbol Device:R
- added R2, R3, R4, R5: 10kΩ, Resistor_SMD:R_0603_1608Metric, symbol Device:R
- added SW1: RESET, Button_Switch_SMD:SW_Tactile_SPST_NO_Straight_CK_PTS636Sx25SMTRLFS, symbol Switch:SW_MEC_5G
- added SW2: WKUP, Button_Switch_SMD:SW_Tactile_SPST_NO_Straight_CK_PTS636Sx25SMTRLFS, symbol Switch:SW_MEC_5G
- added U2: AMS1117-3.3, Package_TO_SOT_SMD:SOT-223-3_TabPin2, symbol Regulator_Linear:AMS1117-3.3
Connections:
- net 3V3 is gone; now on net VCC_3V3: C5.2, C6.2, C7.2, C8.2, D3.1 (VDD), D4.1 (VDD), D7.1 (VDD), D8.1 (VDD)
- net Earth: now also U1.23 (VSS), U1.35 (VSS), U1.47 (VSS), U1.8 (VSSA), C10.2, C11.2, C12.1, C9.2, J1.A1 (GND), J1.A12 (GND), J1.B1 (GND), J1.B12 (GND), J2.1 (Pin_1), R2.1, R4.1, R5.2, SW1.3 (B), SW1.4 (B), U2.1 (GND)
- net VCC_3V3: now also C10.1, C11.1, C9.1, J2.4 (Pin_4), R1.1, R3.2, SW2.3 (B), SW2.4 (B), U2.2 (VO)
- net WKUP: now reaches U1.10 (PA0)
- net WKUP: now also SW2.1 (A), SW2.2 (A)
- net BOOT1/PB2: now reaches U1.20 (PB2)
- net BOOT1/PB2: now also R5.1
- net SWDIO: now reaches U1.34 (PA13)
- net SWDIO: now also J2.3 (Pin_3), R3.1
- net SWCLK: now reaches U1.37 (PA14)
- net SWCLK: now also J2.2 (Pin_2), R2.2
- net LED_IN: now reaches U1.43 (PB7)
- net LED_IN: now also D1.4 (DIN)
- net BOOT0: now reaches U1.44 (BOOT0)
- net BOOT0: now also R4.2
- net RESET: now reaches U1.7 (NRST)
- net RESET: now also C12.2, R1.2, SW1.1 (A), SW1.2 (A)
- new net VCC_5V: J1.A4 (VBUS), J1.A9 (VBUS), J1.B4 (VBUS), J1.B9 (VBUS), U2.3 (VI)

Commit message: three
Parts:
- removed SW1: RESET, Button_Switch_SMD:SW_Tactile_SPST_NO_Straight_CK_PTS636Sx25SMTRLFS, symbol Switch:SW_MEC_5G
- removed SW2: WKUP, Button_Switch_SMD:SW_Tactile_SPST_NO_Straight_CK_PTS636Sx25SMTRLFS, symbol Switch:SW_MEC_5G
- added SW1: RESET, Button_Switch_SMD:SW_Push_1P1T_NO_Vertical_Wuerth_434133025816, symbol Switch:SW_Push_Dual
- added SW2: WKUP, Button_Switch_SMD:SW_Push_1P1T_NO_Vertical_Wuerth_434133025816, symbol Switch:SW_Push_Dual
- J1: footprint (none) -> Connector_USB:USB_C_Receptacle_G-Switch_GT-USB-7010ASV
- renumbered D5 to D2, D2 to D3, D6 to D4, D3 to D5, D7 to D6, D4 to D7
Connections:
- net Earth: now also SW1.2 (4)
- net RESET: now also SW1.1 (2)
- net VCC_3V3: now also SW2.2 (4)
- net WKUP: now also SW2.1 (2)
- net at D7.4 (DIN): now also D6.2 (DOUT)
- no-connect marks 0 -> 46

Commit message: 连线STEP-1
Parts:
- added C13: 100nf, Capacitor_SMD:C_0603_1608Metric, symbol Device:C
- added R6: 4.7kΩ, Resistor_SMD:R_0603_1608Metric, symbol Device:R
- added R7: 1kΩ, Resistor_SMD:R_0603_1608Metric, symbol Device:R_US
- added SW3: SW_Push_Dual, Button_Switch_THT:SW_Tactile_SPST_Angled_PTS645Vx39-2LFS, symbol Switch:SW_Push_Dual
- C12: value 0.1uf -> 100nf
- R1: value 10k -> 10kΩ
Connections:
- net Earth: now also R6.1
- net VCC_3V3: now also C13.2, SW3.2 (4)
- net Button_LED: now reaches U1.32 (PA11)
- net Button_LED: now also R7.2
- new net: C13.1, R6.2, R7.1, SW3.1 (3)
- no-connect marks 46 -> 41

Commit message: Finish All
Connections:
- net Earth: now also J1.S1 (SHIELD)
- net SWCLK: now also J2.3 (Pin_3), R3.1; no longer J2.2 (Pin_2), R2.2
- net SWDIO: now also J2.2 (Pin_2), R2.2; no longer J2.3 (Pin_3), R3.1
- no-connect marks 41 -> 40
Changed lines of the file:
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@@
   (junction (at 201.93 83.82) (diameter 0) (color 0 0 0 0)
+  )
+  (junction (at 49.53 185.42) (diameter 0) (color 0 0 0 0)
   )
   (junction (at 201.93 130.81) (diameter 0) (color 0 0 0 0)
@@
   (no_connect (at 64.77 33.02))
   (no_connect (at 31.75 66.04))
-  (no_connect (at 41.91 176.53))
   (no_connect (at 209.55 92.71))
   (no_connect (at 31.75 58.42))
@@
     (stroke (width 0) (type default))
   )
+  (wire (pts (xy 41.91 185.42) (xy 49.53 185.42))
+    (stroke (width 0) (type default))
+  )
   (wire (pts (xy 204.47 34.29) (xy 222.25 34.29))
     (stroke (width 0) (type default))
@@
   )
   (wire (pts (xy 106.68 34.29) (xy 140.97 34.29))
+    (stroke (width 0) (type default))
+  )
+  (wire (pts (xy 41.91 176.53) (xy 41.91 185.42))
     (stroke (width 0) (type default))
   )
@@
     (effects (font (size 1.27 1.27)) (justify left bottom))
   )
-  (label "SWDIO" (at 119.38 171.45 180) (fields_autoplaced)
+  (label "SWCLK" (at 119.38 171.45 180) (fields_autoplaced)
     (effects (font (size 1.27 1.27)) (justify right bottom))
   )
@@
     (effects (font (size 1.27 1.27)) (justify left bottom))
   )
+  (label "SWDIO" (at 119.38 168.91 180) (fields_autoplaced)
+    (effects (font (size 1.27 1.27)) (justify right bottom))
+  )
   (label "GND" (at 52.07 181.61 0) (fields_autoplaced)
     (effects (font (size 1.27 1.27)) (justify left bottom))
@@
   (label "VCC_3V3" (at 100.33 186.69 90) (fields_autoplaced)
     (effects (font (size 1.27 1.27)) (justify left bottom))
-  )
-  (label "SWCLK" (at 119.38 168.91 180) (fields_autoplaced)
-    (effects (font (size 1.27 1.27)) (justify right bottom))
   )
   (label "VCC_3V3" (at 119.38 107.95 0) (fields_autoplaced)
@@
     )
     (pin "1")
-    (pin "2")
-    (pin "1")
+    (pin "1")
+    (pin "2")
     (pin "2")
     (instances
@@
     )
     (pin "1")
-    (pin "2")
-    (pin "1")
+    (pin "1")
+    (pin "2")
     (pin "2")
     (instances
@@
     )
     (pin "1")
-    (pin "2")
-    (pin "1")
-    (pin "2")
-    (instances
+    (pin "1")
+    (pin "2")
+    (pin "2")
+    (instances

Commit message: 修改-1
Connections:
- net VCC_3V3: no longer C1.2, C2.2, C3.2, C4.2, C5.2, C6.2, C7.2, C8.2, D1.1 (VDD), D2.1 (VDD), D3.1 (VDD), D4.1 (VDD), D5.1 (VDD), D6.1 (VDD), D7.1 (VDD), D8.1 (VDD)
- net VCC_5V: now also C1.2, C2.2, C3.2, C4.2, C5.2, C6.2, C7.2, C8.2, D1.1 (VDD), D2.1 (VDD), D3.1 (VDD), D4.1 (VDD), D5.1 (VDD), D6.1 (VDD), D7.1 (VDD), D8.1 (VDD)
Changed lines of the file:
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@@
-    (effects (font (size 1.27 1.27)) (justify right bottom))
-  )
-  (label "VCC_3V3" (at 222.25 83.82 180) (fields_autoplaced)
     (effects (font (size 1.27 1.27)) (justify right bottom))
   )
@@
     (effects (font (size 1.27 1.27)) (justify left bottom))
   )
-  (label "VCC_3V3" (at 91.44 44.45 0) (fields_autoplaced)
+  (label "LED_IN" (at 91.44 53.34 0) (fields_autoplaced)
     (effects (font (size 1.27 1.27)) (justify left bottom))
   )
-  (label "LED_IN" (at 91.44 53.34 0) (fields_autoplaced)
-    (effects (font (size 1.27 1.27)) (justify left bottom))
+  (label "VCC_5V" (at 222.25 83.82 180) (fields_autoplaced)
+    (effects (font (size 1.27 1.27)) (justify right bottom))
   )
   (label "VCC_3V3" (at 180.34 107.95 0) (fields_autoplaced)
@@
     (effects (font (size 1.27 1.27)) (justify left bottom))
   )
+  (label "VCC_5V" (at 91.44 44.45 0) (fields_autoplaced)
+    (effects (font (size 1.27 1.27)) (justify left bottom))
+  )
