File: RM_47mm.kicad_pcb (KiCad board)
At the start: 4 copper layers, 40 x 40 mm, 37 parts, among them J1 USB_C_Receptacle_USB2.0, J2 SWD, SW1 RESET, SW2 WKUP, SW3 SW_Push_Dual, U1 STM32F103C8Tx, U2 AMS1117-3.3

Commit message: Manufactor
Parts:
- moved G*** 2.95 mm to (163.8, 103.9)
Changed lines of the file:
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@@
   )
   (footprint "Library:QianLi_20mm" (layer "B.Cu")
-    (at 164.565897 101.038431 -90)
+    (at 163.841784 103.903237 -90)
     (attr board_only exclude_from_pos_files exclude_from_bom)
     (fp_text reference "G***" (at 0 0 90) (layer "B.SilkS") hide

Commit message: Finished
Parts:
- SW2: footprint Button_Switch_SMD:SW_Push_1P1T_NO_Vertical_Wuerth_434133025816 -> Library:3.46*3.43*1.5mm push button

Commit message: 修改-1
Parts:
- SW2: footprint Library:3.46*3.43*1.5mm push button -> Button_Switch_SMD:SW_Push_1P1T_NO_Vertical_Wuerth_434133025816
Connections:
- C1 pad 2: /VCC_3V3 -> /VCC_5V
- C2 pad 2: /VCC_3V3 -> /VCC_5V
- C3 pad 2: /VCC_3V3 -> /VCC_5V
- C4 pad 2: /VCC_3V3 -> /VCC_5V
- C5 pad 2: /VCC_3V3 -> /VCC_5V
- C6 pad 2: /VCC_3V3 -> /VCC_5V
- C7 pad 2: /VCC_3V3 -> /VCC_5V
- C8 pad 2: /VCC_3V3 -> /VCC_5V
- D1 pad 1: /VCC_3V3 -> /VCC_5V
- D2 pad 1: /VCC_3V3 -> /VCC_5V
- D3 pad 1: /VCC_3V3 -> /VCC_5V
- D4 pad 1: /VCC_3V3 -> /VCC_5V
- D5 pad 1: /VCC_3V3 -> /VCC_5V
- D6 pad 1: /VCC_3V3 -> /VCC_5V
- D7 pad 1: /VCC_3V3 -> /VCC_5V
- D8 pad 1: /VCC_3V3 -> /VCC_5V
Routing:
- net /VCC_5V: track 18.2 -> 118.9 mm, vias 0 -> 1
- net /VCC_3V3: track 95.5 -> 58.3 mm, vias 11 -> 7

Commit message: Final-3
Routing:
- net Earth: track 102.2 -> 99.8 mm
- net Net-(C1-Pad1): track 48.4 -> 46.1 mm
- net /VCC_5V: track 118.9 -> 120.2 mm
- net /LED_IN: track 11.0 -> 10.2 mm
